File: 20khzActive/filter.sch (KiCad schematic (older format))
At the start: 51 parts, among them J1 in, J2 ut, J3 in, J4 ut, J5 GND_conns, J6 PWR_Ext, U1 NE5532, U2 NE5532, U3 74LVC125, U4 NE5532, U5 NE5532, U6 LM2937

Commit message: 5.0
Parts:
- C1, C10, C11, C12, C13, C14, C15, C16, C17, C18, C19, C2, C20, C21, C22, C23, C3, C4, C5, C6, C7, C8, C9: symbol C -> device:C
- J1, J2, J3, J4, J5, J6: symbol Conn_01x02 -> conn:Conn_01x02
- R1, R10, R11, R12, R13, R14, R15, R16, R2, R3, R4, R5, R6, R7, R8, R9: symbol R -> device:R
- U1, U2, U4, U5: symbol NE5532 -> linear:NE5532
- U3: symbol 74LVC125 -> filter-rescue:74LVC125
- U6: symbol LM2937 -> Peters:LM2937
Connections:
- wire segments 122 -> 149
